File: Solar Cell offgrid Power.kicad_pcb (KiCad board)
At the start: 2 copper layers, 124.5 x 68.1 mm, 14 parts, among them J1 Conn_01x10_Socket, J2 Conn_01x10_Pin, J3 Screw_Terminal_01x02, Q1 S8550

Commit message: Add files via upload
Parts:
- removed BT3: BK-18650-PC4, Battery:2x 18650 Battery holder BAT_BK-18650-PC4
- removed S1: MHSS1104, Button_Switch_THT:Toggle Switch 2 pos PCB MSS-22D18G2 2P2T
- added BK1: Copper Track Breaker, AeonLabs_Connectors:Copper Track Breaker 2 points, F.Cu at (175.0, 111.9)
- added BK2: Copper Track Breaker, AeonLabs_Connectors:Copper Track Breaker 2 points, F.Cu at (178.1, 111.9)
- added BK3: Copper Track Breaker, AeonLabs_Connectors:Copper Track Breaker 2 points, F.Cu at (181.1, 111.9)
- added BK4: Copper Track Breaker, AeonLabs_Connectors:Copper Track Breaker 2 points, F.Cu at (160.6, 112.0)
- added BK5: Copper Track Breaker, AeonLabs_Connectors:Copper Track Breaker 2 points, F.Cu at (163.3, 112.0)
- added BK6: Copper Track Breaker, AeonLabs_Connectors:Copper Track Breaker 2 points, F.Cu at (166.0, 112.0)
- added BK7: Copper Track Breaker, AeonLabs_Connectors:Copper Track Breaker 2 points, F.Cu at (168.9, 111.9)
- added BK8: Copper Track Breaker, AeonLabs_Connectors:Copper Track Breaker 2 points, F.Cu at (172.0, 111.9)
- added BT2: BK-18650-PC4, Battery:2x 18650 Battery holder BAT_BK-18650-PC4, F.Cu at (172.1, 86.9)
- added G***: LOGO, AeonLabs Logos:smart build design, F.Cu at (122.6, 129.1)
- added J4: Conn_02x03_Counter_Clockwise, Button_Switch_THT:Toggle Switch 2 pos PCB MSS-22D18G2 2P2T, F.Cu at (124.3, 132.2)
- added REF**: OSHW-Logo2_14.6x12mm_SilkScreen, Symbol:OSHW-Logo2_14.6x12mm_SilkScreen, F.Cu at (217.5, 123.0)
- G***, REF**: moved to B.Cu
- moved REF** 36.2 mm to (158.1, 104.5), turned to 180 degrees
- moved G*** 23.7 mm to (179.7, 104.5), turned to 180 degrees
- moved R1 7.55 mm to (128.0, 93.4), turned to 0 degrees
- moved Q1 4.15 mm to (121.8, 88.4)
- moved D1 3.64 mm to (128.1, 89.6)
- moved BAT_POS2 3.48 mm to (131.2, 77.1)
- moved TPBAT_NEG1 2.81 mm to (213.6, 76.3)
Connections:
- J1 pad 1: unconnected-(J1-Pin_1-Pad1) -> Conn_track_1
- J1 pad 10: unconnected-(J1-Pin_10-Pad10) -> Conn_track_10
- J1 pad 2: unconnected-(J1-Pin_2-Pad2) -> Conn_track_2
- J1 pad 3: unconnected-(J1-Pin_3-Pad3) -> Conn_track_3
- J1 pad 4: PWR -> Conn_track_4
- J1 pad 7: GND -> Conn_track_7
- J1 pad 8: unconnected-(J1-Pin_8-Pad8) -> Conn_track_8
- J1 pad 9: unconnected-(J1-Pin_9-Pad9) -> Conn_track_9
- J2 pad 1: unconnected-(J2-Pin_1-Pad1) -> Conn_track_1
- J2 pad 10: unconnected-(J2-Pin_10-Pad10) -> Conn_track_10
- J2 pad 2: unconnected-(J2-Pin_2-Pad2) -> Conn_track_2
- J2 pad 3: unconnected-(J2-Pin_3-Pad3) -> Conn_track_3
- J2 pad 4: PWR -> Conn_track_4
- J2 pad 7: GND -> Conn_track_7
- J2 pad 8: unconnected-(J2-Pin_8-Pad8) -> Conn_track_8
- J2 pad 9: unconnected-(J2-Pin_9-Pad9) -> Conn_track_9
Routing:
- net Conn_track_10: track 0.00 -> 135.1 mm, vias 0 -> 1
- net Conn_track_9: track 0.00 -> 131.9 mm, vias 0 -> 1
- net Conn_track_8: track 0.00 -> 131.1 mm, vias 0 -> 1
- net Conn_track_7: track 0.00 -> 131.0 mm, vias 0 -> 1
- net Conn_track_4: track 0.00 -> 118.8 mm, vias 0 -> 1
- net Conn_track_3: track 0.00 -> 116.3 mm, vias 0 -> 1
- net Conn_track_2: track 0.00 -> 115.6 mm, vias 0 -> 1
- net Conn_track_1: track 0.00 -> 115.4 mm, vias 0 -> 1
- net BAT+: track 49.7 -> 134.3 mm, vias 0 -> 2
- net GND: track 301.2 -> 276.9 mm
- net Net-(D1-A): track 128.6 -> 117.1 mm
- net Net-(S1-Pad5): track 9.16 -> 0.00 mm
- net PWR: track 190.7 -> 196.6 mm
- net Net-(J4-Pin_1): track 0.00 -> 5.64 mm
- net Net-(Q1-B): track 12.9 -> 14.9 mm
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Other:
- board text added: "1"
- board text added: "10"
- board text added: "2"
- board text added: "3"
- board text added: "4"
- board text added: "7"
- board text added: "8"
- board text added: "9"
- board text added: "Battery Channel IO"
- board text added: "FOR SINGLE BLUE SOLAR TILE 2x 18650 liPo BATTERY"
- board text added: "POWER"
- board text added: "make sure you have a unique channel number on the rail"
